File: Smart_Project.kicad_pcb (KiCad board)
At the start: 2 copper layers, 68.6 x 53.3 mm, 24 parts, among them P1 Power, P2 Analog, P3 Digital, P4 Digital, P5 CONN_01X01, P6 CONN_01X01, P7 CONN_01X01, P8 CONN_01X01, U1 LTC1050, U2 LTC1050

Commit message: Modification des largeurs de pistes et ajout du plan de masse
Parts:
- moved R6 14.6 mm to (123.4, 109.7), turned to 90 degrees
Routing:
- net GND: track 122.7 -> 0.00 mm, vias 2 -> 0
- net Comparateur_Output: track 0.00 -> 85.0 mm, vias 0 -> 4
- net A0: track 16.2 -> 80.0 mm, vias 0 -> 2
- net +3V3: track 47.8 -> 61.8 mm
- net Net-(C4-Pad1): track 29.4 -> 39.2 mm
- net +5V: track 32.7 -> 39.6 mm
- net Net-(RA1-Pad1): track 11.3 -> 13.3 mm
- net Net-(C4-Pad2): track 17.0 -> 18.8 mm
- added copper zone on B.Cu, net GND
Other:
- net class Alim added: clearance 0.5, trace_width 0.8, via_dia 1.8, via_drill 0.8
- net class Default: clearance 0.2 -> 0.5; trace_width 0.25 -> 0.5; via_dia 0.6 -> 1.8; via_drill 0.4 -> 0.8
- rule trace_clearance: 0.2 -> 0.5
- board text added: "R.Rodriguez J.Vincent 5ISS 2019"
